File: Hardware/Bottom/Orion-BOTTOM.sch (EAGLE design)
At the start: 0 parts

Commit message: fixed some missing design blocks
Parts:
- added C10, C11, C17, C18, C22, C24: 100n, LinnesLab-Passives:CAPACITOR0603
- added C14, C19: 2.2n, LinnesLab-Passives:CAPACITOR0603
- added C15, C16: 2.2u, LinnesLab-Passives:CAPACITOR0603
- added C20: 22u, LinnesLab-Passives:CAPACITOR0603
- added C21: 22n, LinnesLab-Passives:CAPACITOR0603
- added IMU1: LSM6DS3_CAST, LinnesLab-Sensors:LSM6DS3_CAST
- added J1: (no value), LinnesLab-Connectors:CONN_07
- added OP3: (no value), LinnesLab-AnalogIC:OP-QUAD-SO14
- added OP4: (no value), LinnesLab-AnalogIC:OP-SINGLEOT
- added Q1: (no value), LinnesLab-DiscreteSemi:NPN-GENERIC
- added R13, R15, R19, R21: 220k, LinnesLab-Passives:RESISTOR0603
- added R14, R22: 10M, LinnesLab-Passives:RESISTOR0603
- added R16: (no value), LinnesLab-Passives:RESISTOR0603
- added R17, R18: 10k, LinnesLab-Passives:RESISTOR0402
- added R20, R23: 1M, LinnesLab-Passives:RESISTOR0603
- added R24: 10k, LinnesLab-Passives:RESISTOR0603
- added U$3: (no value), LinnesLab-Connectors:PPG.MODULE.2
- added U$4: AD5171, LinnesLab-DigitalIC:AD5171
- added U1: AD5242-SO16, LinnesLab-DigitalIC:AD5242-SO16
Connections:
- new net 3.3V: C11.2, C17.2, C18.2, C22.2, C24.2, IMU1.VCC, OP3G$5.V+, OP4G$2.V+, R13.2, R15.2, R17.2, U$3.V+, U$4.A0, U$4.VDD, U1.!SHDN, U1.VDD
- new net G.A1: U1.A1
- new net G.A2: U1.A2
- new net G.O1: U1.O1
- new net G.O2: U1.O2
- new net G.W2: C21.1, OP3G$1.-IN, R24.1, U1.W2
- new net GND: C11.1, C17.1, C18.1, C22.1, C24.1, IMU1.GND, OP3G$5.V-, OP4G$1.+IN, OP4G$2.V-, Q1.E, R18.1, R19.1, R21.1, U$3.GND, U$4.GND, U1.AD0, U1.AD1, U1.DGND, U1.VSS
- new net LED: Q1.C
- new net LED.C: U$3.LD1.C
- new net LED.CTRL: U$4.A
- new net N$10: OP3G$4.+IN, R17.1, R18.2
- new net N$13: C15.2, OP3G$2.+IN, R13.1, R19.2
- new net N$15: C14.2, OP3G$2.-IN, R14.1, R20.2
- new net N$16: C14.1, C16.1, OP3G$2.OUT, R14.2
- new net N$17: C16.2, OP3G$3.+IN, R15.1, R21.2
- new net N$18: C19.2, OP3G$3.-IN, R22.1, R23.2
- new net N$19: C19.1, C20.1, OP3G$3.OUT, R22.2
- new net N$20: C20.2, R24.2
- new net N$8: Q1.B, R16.2
- new net N$9: R16.1, U$4.B, U$4.W
- new net PD.C: C10.1, OP4G$1.-IN, U$3.PD.C, U1.B1
- new net PPG: C21.2, OP3G$1.OUT, U1.B2
- new net SCL: IMU1.SCL, U$4.SCL, U1.SCL
- new net SDA: IMU1.SDA, U$4.SDA, U1.SDA
- new net TIA: C10.2, C15.1, OP4G$1.OUT, U1.W1
- new net VREF: OP3G$1.+IN, OP3G$4.-IN, OP3G$4.OUT, R20.1, R23.1
Other:
- note added: "Active Bandpass Filters"
- note added: "Digital Potentiometers"
- note added: "I2C Address: 0x2C"
- note added: "I2C Address: 0x2D"
- note added: "Photodiode and LEDs"
- note added: "Transimpedance Amplifier"
