File: Hardware/Top/Orion-TOP.sch (EAGLE design)
At the start: 49 parts, among them U2 NRF52832_MODULE_MDBT42, U5 PCF8523

Commit message: modified top board schemetics: add buttons and organized
Parts:
- removed C14: 100n, LinnesLab-Passives:CAPACITOR0603
- removed D1: (no value), LinnesLab-DiscreteSemi:SCHOTTKY-USC
- removed R5: 10k, LinnesLab-Passives:RESISTOR0603
- added SW1, SW2, SW5: SWITCH.MOM, LinnesLab-Switches:SWITCH.MOM
Connections:
- removed net DTR: C14.1
- new net SW1: SW1.1, SW2.1, SW5.1
- net 3.3V: no longer D1.C, R5.2
- net GND: now also SW1.3, SW1.4, SW2.3, SW2.4, SW5.3, SW5.4
- net RESET: no longer C14.2, D1.A, R5.1
Other:
- note added: "Buttons"
- note added: "Cortex Debugger/ Programmer"
- note added: "Power Management"
- note added: "Real-Time Clock"
- note added: "SD Card"
- note added: "nRF52832 Module"
- note removed: "100nF+10K @ 3.3V = ~1.2ms to 0.7VCC"
- note removed: "Microcontroller Reset Circuit"
- moved on the sheet: C10, C11, C12, C20, C21, C22, C5, C6, C7, C8, C9, CHRG2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

Commit message: fixed some missing design blocks
Parts:
- added C14, C23: 47p, LinnesLab-Passives:CAPACITOR0603
- added C31, C4: 100n, LinnesLab-Passives:CAPACITOR0603
- added D1: (no value), LinnesLab-DiscreteSemi:SCHOTTKY-USC
- added J1: (no value), LinnesLab-Connectors:CONN_07
- added J3: (no value), LinnesLab-Connectors:CONN_061.27MM
- added JP2: (no value), LinnesLab-Switches:JUMPER-SMT_2_NO_SILK
- added LED5: RED, LinnesLab-LED:LED0603
- added LED6: YELLOW, LinnesLab-LED:LED0603
- added R17: 10k, LinnesLab-Passives:RESISTOR0603
- added R18, R9: 27, LinnesLab-Passives:RESISTOR0603
- added R19, R20: 1k, LinnesLab-Passives:RESISTOR0603
- added SW9: (no value), LinnesLab-Switches:SPST-PTS830GG140-COPY.1-3
- added U4: FT231XS, LinnesLab-DigitalIC:FT231XS
- added USB3: USB.MICRO-BIGGERPADS, LinnesLab-Connectors:USB.MICRO-BIGGERPADS
- XTAL3: FREQ 32.7680KHZ -> (none)
Connections:
- removed net BATT: R13.1, R14.2
- removed net CHRG.STAT: CHRG2.STAT, R12.1
- removed net SD.CS: SD2.CS
- new net !CTS: JP2.2, U4.!CTS
- new net !DTR: U4.!DTR
- new net A4/BATT: R13.1, R14.2, U2.P0.28/AIN4
- new net D11/SW1: SW1.1, U2.P0.11
- new net D15/SW2: SW2.1, U2.P0.15
- new net D27/CHRG.STATUS: CHRG2.STAT, R12.1, U2.P0.27
- new net D7/SD.CS: SD2.CS, U2.P0.07
- new net DTR: C31.1
- new net FT3V3: U4.3V3OUT
- new net N$23: R9.2, U4.USBDM
- new net N$24: R18.2, U4.USBDP
- new net N$25: LED5.C, R19.2
- new net N$26: LED6.C, R20.2
- new net RXLED: R19.1, U4.CBUS1
- new net TXLED: R20.1, U4.CBUS2
- new net USB_D+: C14.1, R18.1, USB3.D+
- new net USB_D-: C23.2, R9.1, USB3.D-
- net 3.3V: now also C4.2, D1.C, LED5.A, LED6.A, R17.2, U4.!RESET, U4.VCCIO
- net GND: now also C14.2, C23.1, C4.1, JP2.1, SW9.B, U4.GND@16, U4.GND@6, USB3.GND, USB3.SHIELD
- net RESET: now also C31.2, D1.A, R17.1, SW9.A
- net RXD: now also U4.RXD
- net SW1: no longer SW1.1, SW2.1
- net TXD: now also U4.TXD
- net V_USB: now also U4.VCC, USB3.V+
Other:
- note added: "100nF+10K @ 3.3V = ~1.2ms to 0.7VCC"
- note added: "I don't remember if CTS needs to be grounded or left floating so here's a jumper to ground so it can be configued either way dynamically."
- note added: "Microcontroller Reset Circuit"
- note added: "TXD goes to RX on the other device RXD goes to TX on the other device"
